File: Prototype2/schematic/Prototype2.sch (KiCad schematic (older format))
At the start: 4 parts, among them U1 HD63C09E, U2 628128, U3 ATtiny85-20PU

Commit message: Introduce 0-LocalLibrary to Prototype1 and 2
Parts:
- U1: footprint Package_DIP:DIP-40_W15.24mm -> Package_DIP:DIP-40_W15.24mm_Socket
- U2: footprint (none) -> Package_DIP:DIP-32_W15.24mm_Socket; symbol Memory_RAM:628128 -> 0-LocalLibrary:628128
- U3: symbol MCU_Microchip_ATtiny:ATtiny85-20PU -> 0-LocalLibrary:ATtiny85-20PU
Connections:
- net labels added: ~ACK, ~HALT, ~INT, ~RAM_E, ~RESET, ~STEP
- net labels removed: #ACK, #HALT, #RESET, #STEP, RAM_E
- wire segments 83 -> 98
