File: BionicBase/schematic-teensy35-breadboard/Prototype1.kicad_pcb (KiCad board)
At the start: 2 copper layers, 13 parts, among them J5 Conn_01x24_T1-T24_30_53, J6 Conn_01x20_T1-T20_34_53, J7 Conn_01x20_T21-T40_34_53, J8 ZIF_Socket_48pin, J9 Conn_01x24_T25-T48_30_53, SW1 Tact_SW, U1 74HCT126

Commit message: Migrate to KiCad 6.0
Other:
- net class Default removed
