File: BionicBase/schematic-teensy35-breadboard/Prototype1.kicad_sch (KiCad schematic)
At the start: 17 parts, among them J1 Conn_01x24_Teensy35_Bionic_1-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, J2 Conn_01x24_Teensy35_Bionic_25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, J3 Conn_01x07_HCT126_1-7_57-63, J4 Conn_01x07_HCT126_8-14_57-63, J5 Conn_01x24_T1-T24_30_53, J6 Conn_01x20_T1-T20_34_53, J7 Conn_01x20_T21-T40_34_53, J8 ZIF_Socket_48pin, J9 Conn_01x24_T25-T48_30_53, SW1 Tact_SW, U1 74HCT126

Commit message: Satisfy Electrical Rules Checker
Other:
- moved on the sheet: J1, J2, J5, J6, J7, J8, J9, Jj5
