File: BionicNS32016/schematic/Prototype1.kicad_pcb (KiCad board)
At the start: 2 copper layers, 66 x 71.1 mm, 15 parts, among them J1 BionicConnector, U1 NS32016N, U2 74HCT126, U3 74HCT541, U4 74HCT541

Commit message: Migrate to KiCad 6.0
Other:
- net class Default removed
