File: BionicP8048/schematic/Prototype1.kicad_pcb (KiCad board)
At the start: 2 copper layers, 48.3 x 71.1 mm, 8 parts, among them J1 BionicConnector, U1 MSM80C39RS, U2 74HCT126

Commit message: Migrate to KiCad 6.0
Other:
- net class Default removed
