File: BionicP8095/schematic/Prototype1.kicad_pcb (KiCad board)
At the start: 2 copper layers, 48.3 x 83.8 mm, 8 parts, among them J1 BionicConnector, U1 P8095BH, U2 74HCT126

Commit message: Migrate to KiCad 6.0
Other:
- net class Default removed
