File: BionicBase/schematic-teensy35/Prototype1.kicad_sch (KiCad schematic)
At the start: 6 parts, among them J1 Bionic_ZIF_Socket_48pin, SW1 Tact_SW

Commit message: Satisfy Electrical Rules Checker
Changed lines of the file:
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@@
+    (effects (font (size 1.27 1.27)) (justify left bottom))
+  )
+  (label "P3[0..7]" (at 78.74 46.99 0)
     (effects (font (size 1.27 1.27)) (justify left bottom))
   )
@@
     (effects (font (size 1.27 1.27)) (justify left bottom))
   )
+  (label "P5[0..7]" (at 78.74 132.08 0)
+    (effects (font (size 1.27 1.27)) (justify left bottom))
+  )
   (label "P10" (at 151.13 60.96 0)
     (effects (font (size 1.27 1.27)) (justify left bottom))
@@
     (effects (font (size 1.27 1.27)) (justify right bottom))
   )
+  (label "P4[0..7]" (at 104.14 86.36 0)
+    (effects (font (size 1.27 1.27)) (justify left bottom))
+  )
   (label "P46" (at 92.71 107.95 0)
     (effects (font (size 1.27 1.27)) (justify left bottom))
@@
     (effects (font (size 1.27 1.27)) (justify left bottom))
   )
+  (label "P1[0..7]" (at 78.74 49.53 0)
+    (effects (font (size 1.27 1.27)) (justify left bottom))
+  )
   (label "P57" (at 92.71 123.19 0)
     (effects (font (size 1.27 1.27)) (justify left bottom))
@@
     (effects (font (size 1.27 1.27)) (justify right bottom))
   )
+  (label "P2[0..7]" (at 105.41 52.07 0)
+    (effects (font (size 1.27 1.27)) (justify left bottom))
+  )
   (label "P54" (at 92.71 115.57 0)
     (effects (font (size 1.27 1.27)) (justify left bottom))
@@
   (label "P25" (at 151.13 96.52 0)
     (effects (font (size 1.27 1.27)) (justify left bottom))
-  )
-  (symbol (lib_id "power:VCC") (at -1352.55 -1136.65 0) (unit 1)
-    (in_bom yes) (on_board yes)
-    (property "Reference" "#PWR01" (id 0) (at -1352.55 -1132.84 0)
-      (effects (font (size 1.27 1.27)) hide)
-    )
-    (property "Value" "VCC" (id 1) (at -1352.1182 -1141.0442 0))
-    (property "Footprint" "" (id 2) (at -1352.55 -1136.65 0)
-      (effects (font (size 1.27 1.27)) hide)
-    )
-    (property "Datasheet" "" (id 3) (at -1352.55 -1136.65 0)
-      (effects (font (size 1.27 1.27)) hide)
-    )
-    (pin "1")
   )
   (symbol (lib_id "power:VCC") (at 120.65 119.38 0) (unit 1)
@@
   (symbol (lib_id "power:+3.3V") (at 100.33 154.94 0) (unit 1)
     (in_bom yes) (on_board yes)
-    (property "Reference" "#PWR?" (id 0) (at 100.33 158.75 0)
+    (property "Reference" "#PWR0102" (id 0) (at 100.33 158.75 0)
       (effects (font (size 1.27 1.27)) hide)
     )
@@
   )
   (symbol_instances
-    (path "/00000000-0000-0000-0000-00005cde46a4"
-      (reference "#PWR01") (unit 1) (value "VCC") (footprint "")
-    )
     (path "/00000000-0000-0000-0000-00005ce5efde"
       (reference "#PWR02") (unit 1) (value "VCC") (footprint "")
@@
     )
     (path "/00000000-0000-0000-0000-0000618a0b8b"
-      (reference "#PWR?") (unit 1) (value "+3.3V") (footprint "")
+      (reference "#PWR0102") (unit 1) (value "+3.3V") (footprint "")
     )
     (path "/00000000-0000-0000-0000-000061858745"
