File: BionicINS8070/schematic/Prototype1.kicad_sch (KiCad schematic)
At the start: 4 parts, among them J1 BionicConnector, U1 INS8070, U2 74HCT126

Commit message: Satisfy Electrical Rules Checker
Other:
- moved on the sheet: U2
