File: BionicMC68008/schematic/Prototype1.kicad_sch (KiCad schematic)
At the start: 9 parts, among them J1 BionicConnector, U1 MC68008P, U2 74HCT126, U3 74HCT541, U4 74HCT541

Commit message: Satisfy Electrical Rules Checker
Other:
- moved on the sheet: C2, U2
