File: BionicMC6809/schematic/Prototype1.kicad_sch (KiCad schematic)
At the start: 5 parts, among them J1 BionicConnector, U1 MC6809P, U2 74HCT126

Commit message: Satisfy Electrical Rules Checker
Other:
- moved on the sheet: U2
