File: BionicNSC800/schematic/Prototype1.kicad_sch (KiCad schematic)
At the start: 4 parts, among them J1 BionicConnector, U1 NSC800N, U2 74HCT126

Commit message: Satisfy Electrical Rules Checker
Other:
- moved on the sheet: C1, J1, U1
